Commit message: Driving Your Virtual Robot
Driving Your Virtual Robot

File: description/robot_core.xacro (robot description, xacro)
@@ -41,4 +41,7 @@
         <origin xyz = "-0.1 0 0"/>
     </joint>
+    <gazebo reference = "chassis">
+        <material>Gazebo/White</material>
+    </gazebo>
     <!-- LEFT WHEEL LINK -->
     <link name = "left_wheel">
@@ -64,4 +67,7 @@
         <axis xyz = "0 0 1"/>
     </joint>
+    <gazebo reference = "left_wheel">
+        <material>Gazebo/Blue</material>
+    </gazebo>
     <!-- RIGHT WHEEL LINK -->
     <link name = "right_wheel">
@@ -87,4 +93,7 @@
         <axis xyz = "0 0 -1"/>
     </joint>
+    <gazebo reference = "right_wheel">
+        <material>Gazebo/Blue</material>
+    </gazebo>
     <!-- CASTER WHEEL LINK -->
     <link name = "caster_wheel">
@@ -109,4 +118,9 @@
         <origin xyz = "0.24 0 0"/>
     </joint>
+    <gazebo reference = "caster_wheel">
+        <material>Gazebo/Black</material>
+        <mu1 value = "0.001"/>
+        <mu2 value = "0.001"/>
+    </gazebo>
 </robot>
 <!-- FOR CONTINUOUS GUI -->
